File: pcb/loco.kicad_pcb (KiCad board)
At the start: 4 copper layers, 69.5 x 29.3 mm, 85 parts, among them J1 POWER, J2 INPUT, J3 I2C, J4 UART, J5 TagConnect, J6 GPIO_A, J7 GPIO_B, J8 Motor1, J9 Motor2, U1 NCV8718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

Commit message: BSP
Parts:
- C10, C11, C6, C7: value C -> 22nF
- C5, C8, C9: value C -> 1uF
- R1, R11, R12, R24, R26: value R -> 10KΩ
- R17, R19: value R -> 15KΩ
- R18, R20, R27, R28, R6: value R -> 1KΩ
- R2, R3: value R -> 4.7KΩ
- R31, R32: value R -> 47KΩ
Connections:
- RN1 pad 1: /ENC2 -> /ENC1
- RN1 pad 2: /ENC1 -> /ENC2
- U2 pad 18: /ENC2 -> /ENC1
- U2 pad 19: /ENC1 -> /ENC2
