File: pcb/loco.kicad_pcb (KiCad board)
At the start: 4 copper layers, 69.5 x 29.3 mm, 85 parts, among them J1 POWER, J2 INPUT, J3 I2C, J4 UART, J5 TagConnect, J6 GPIO_A, J7 GPIO_B, J8 Motor1, J9 Motor2, U1 NCV8718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

Commit message: pcb rev 0.2
Parts:
- added FB7: DNP, Resistor_SMD:R_0603_1608Metric, F.Cu at (117.1, 55.8)
- added FB8: DNP, Resistor_SMD:R_0603_1608Metric, F.Cu at (101.6, 55.8)
- J1: footprint Connector_JST:JST_SH_BM02B-SRSS-TB_1x02-1MP_P1.00mm_Vertical -> Connector_PinHeader_2.54mm:PinHeader_1x02_P2.54mm_Vertical
- J3, J4: footprint Connector_JST:JST_SH_BM04B-SRSS-TB_1x04-1MP_P1.00mm_Vertical -> Connector_JST:JST_SH_SM04B-SRSS-TB_1x04-1MP_P1.00mm_Horizontal
- moved FB3 6.77 mm to (131.5, 69.8), turned to 180 degrees
- moved R2 4.67 mm to (127.9, 63.5)
- moved FB4 4.00 mm to (128.0, 73.7), turned to 90 degrees
- moved R3 2.00 mm to (127.9, 65.2)
- moved REF** 1.57 mm to (99.8, 56.3)
- moved J1 1.57 mm to (71.2, 68.8), turned to 180 degrees
- moved J4 1.01 mm to (123.2, 75.9), turned to 0 degrees
- moved J3 0.77 mm to (133.3, 65.0), turned to 90 degrees
Routing:
- net VCC: track 13.0 -> 35.7 mm, vias 8 -> 10
- net /GPIO_A_VDD: track 2.46 -> 13.2 mm
- net /GPIO_B_VDD: track 2.46 -> 12.4 mm
- net /UART_VDD: track 2.40 -> 7.30 mm
- net Net-(J3-Pin_3): track 16.6 -> 12.1 mm
- net /I2C_VDD: track 2.41 -> 5.64 mm
- net Net-(J3-Pin_4): track 11.0 -> 12.9 mm
- net Net-(J4-Pin_4): track 8.12 -> 9.92 mm
- net Net-(J4-Pin_3): track 6.92 -> 5.25 mm
- net VDD: track 38.7 -> 38.0 mm, vias 22 -> 23
Other:
- board text added: "- VCC +"
- board text added: "vitaly.codes/loco rev 0.2"
- board text removed: "POWER"
- board text removed: "vitaly.codes/loco rev 0.1"
