File: pcb/loco.kicad_sch (KiCad schematic)
At the start: 84 parts

Commit message: BSP
Connections:
- net ENC1: now also RN.1 (R1.1), U.18 (PA8); no longer RN.2 (R2.1), U.19 (PA9)
- net ENC2: now also RN.2 (R2.1), U.19 (PA9); no longer RN.1 (R1.1), U.18 (PA8)
