File: pcb/loco.kicad_sch (KiCad schematic)
At the start: 84 parts

Commit message: pcb rev 0.2
Parts:
- added FB (x2): FerriteBead, symbol Device:FerriteBead
Connections:
- net GPIO_A_VDD: now also FB.1
- net GPIO_B_VDD: now also FB.1
- net VCC: now also FB.2, FB.2

Commit message: fix pull-down for spi flash
Connections:
- net GND: now also RN.6 (R3.2)
- net VDD: no longer RN.6 (R3.2)
Changed lines of the file:
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@@
   (junction (at 129.54 74.93) (diameter 0) (color 0 0 0 0)
   )
-  (junction (at 157.48 161.29) (diameter 0) (color 0 0 0 0)
-  )
   (junction (at 160.02 161.29) (diameter 0) (color 0 0 0 0)
   )
@@
     (stroke (width 0) (type default))
   )
+  (polyline (pts (xy 28.3464 33.7566) (xy 237.49 33.7566))
+    (stroke (width 0.3) (type dash))
+  )
   (wire (pts (xy 63.5 172.72) (xy 76.2 172.72))
     (stroke (width 0) (type default))
@@
     (stroke (width 0) (type default))
   )
-  (polyline (pts (xy 28.575 144.8816) (xy 236.855 144.8816))
-    (stroke (width 0.3) (type dash))
-  )
   (wire (pts (xy 148.59 105.41) (xy 134.62 105.41))
     (stroke (width 0) (type default))
@@
     (stroke (width 0) (type default))
   )
+  (polyline (pts (xy 237.49 130.175) (xy 28.3464 130.175))
+    (stroke (width 0.3) (type dash))
+  )
   (wire (pts (xy 311.15 88.9) (xy 318.77 88.9))
     (stroke (width 0) (type default))
@@
     (stroke (width 0) (type default))
   )
-  (polyline (pts (xy 28.3464 33.8582) (xy 28.3464 130.2766))
-    (stroke (width 0.3) (type dash))
-  )
   (wire (pts (xy 271.78 67.31) (xy 267.97 67.31))
     (stroke (width 0) (type default))
   )
-  (polyline (pts (xy 28.3464 33.7566) (xy 237.49 33.7566))
-    (stroke (width 0.3) (type dash))
-  )
   (wire (pts (xy 287.02 49.53) (xy 287.02 55.88))
     (stroke (width 0) (type default))
@@
     (stroke (width 0) (type default))
   )
+  (polyline (pts (xy 388.5184 129.9464) (xy 253.0348 129.9464))
+    (stroke (width 0.3) (type dash))
+  )
   (wire (pts (xy 287.02 161.29) (xy 287.02 167.64))
     (stroke (width 0) (type default))
@@
     (stroke (width 0) (type default))
   )
+  (wire (pts (xy 144.145 177.8) (xy 144.145 168.275))
+    (stroke (width 0) (type default))
+  )
   (wire (pts (xy 302.26 73.66) (xy 318.77 73.66))
     (stroke (width 0) (type default))
   )
-  (polyline (pts (xy 236.855 241.3) (xy 28.575 241.3))
+  (polyline (pts (xy 253.0348 145.288) (xy 388.5184 145.288))
+    (stroke (width 0.3) (type dash))
+  )
+  (polyline (pts (xy 388.5184 241.7064) (xy 253.0348 241.7064))
     (stroke (width 0.3) (type dash))
   )
@@
     (stroke (width 0) (type default))
   )
+  (wire (pts (xy 157.48 168.275) (xy 157.48 170.18))
+    (stroke (width 0) (type default))
+  )
   (wire (pts (xy 316.23 228.6) (xy 311.15 228.6))
     (stroke (width 0) (type default))
@@
     (stroke (width 0) (type default))
   )
+  (polyline (pts (xy 237.49 33.7566) (xy 237.49 130.175))
+    (stroke (width 0.3) (type dash))
+  )
   (wire (pts (xy 283.21 116.84) (xy 293.37 116.84))
     (stroke (width 0) (type default))
@@
     (stroke (width 0) (type default))
   )
-  (wire (pts (xy 111.76 161.29) (xy 157.48 161.29))
-    (stroke (width 0) (type default))
-  )
   (wire (pts (xy 283.21 116.84) (xy 283.21 118.11))
     (stroke (width 0) (type default))
@@
     (stroke (width 0) (type default))
   )
+  (polyline (pts (xy 28.3464 33.8582) (xy 28.3464 130.2766))
+    (stroke (width 0.3) (type dash))
+  )
   (wire (pts (xy 138.43 102.87) (xy 138.43 77.47))
     (stroke (width 0) (type default))
@@
     (stroke (width 0) (type default))
   )
+  (polyline (pts (xy 28.575 144.8816) (xy 236.855 144.8816))
+    (stroke (width 0.3) (type dash))
+  )
   (wire (pts (xy 276.86 67.31) (xy 271.78 67.31))
     (stroke (width 0) (type default))
@@
     (stroke (width 0) (type default))
   )
-  (polyline (pts (xy 28.575 145.5166) (xy 28.575 241.935))
-    (stroke (width 0.3) (type dash))
-  )
   (wire (pts (xy 195.58 99.06) (xy 195.58 101.6))
     (stroke (width 0) (type default))
@@
     (stroke (width 0) (type default))
   )
-  (wire (pts (xy 160.02 161.29) (xy 157.48 161.29))
+  (wire (pts (xy 144.145 168.275) (xy 157.48 168.275))
+    (stroke (width 0) (type default))
+  )
+  (wire (pts (xy 111.76 161.29) (xy 160.02 161.29))
     (stroke (width 0) (type default))
   )
@@
     (stroke (width 0) (type default))
   )
+  (polyline (pts (xy 253.0348 33.6296) (xy 253.0348 130.048))
+    (stroke (width 0.3) (type dash))
+  )
   (wire (pts (xy 162.56 190.5) (xy 163.83 190.5))
     (stroke (width 0) (type default))
@@
     (stroke (width 0) (type default))
   )
-  (polyline (pts (xy 253.0348 145.288) (xy 388.5184 145.288))
-    (stroke (width 0.3) (type dash))
-  )
   (wire (pts (xy 283.21 195.58) (xy 283.21 200.66))
     (stroke (width 0) (type default))
@@
     (stroke (width 0) (type default))
   )
-  (polyline (pts (xy 253.0348 33.6296) (xy 253.0348 130.048))
-    (stroke (width 0.3) (type dash))
-  )
   (wire (pts (xy 311.15 96.52) (xy 311.15 99.06))
     (stroke (width 0) (type default))
@@
     (stroke (width 0) (type default))
   )
+  (polyline (pts (xy 253.0348 145.3896) (xy 253.0348 241.808))
+    (stroke (width 0.3) (type dash))
+  )
   (wire (pts (xy 283.21 228.6) (xy 283.21 229.87))
     (stroke (width 0) (type default))
@@
     (stroke (width 0) (type default))
   )
-  (wire (pts (xy 157.48 161.29) (xy 157.48 170.18))
-    (stroke (width 0) (type default))
-  )
   (wire (pts (xy 69.85 73.66) (xy 69.85 69.85))
     (stroke (width 0) (type default))
   )
+  (polyline (pts (xy 388.5184 145.288) (xy 388.5184 241.7064))
+    (stroke (width 0.3) (type dash))
+  )
   (wire (pts (xy 359.41 187.96) (xy 359.41 190.5))
     (stroke (width 0) (type default))
@@
     (stroke (width 0) (type default))
   )
-  (polyline (pts (xy 253.0348 33.528) (xy 388.5184 33.528))
-    (stroke (width 0.3) (type dash))
-  )
   (wire (pts (xy 293.37 228.6) (xy 302.26 228.6))
     (stroke (width 0) (type default))
@@
     (stroke (width 0) (type default))
   )
-  (polyline (pts (xy 237.49 33.7566) (xy 237.49 130.175))
-    (stroke (width 0.3) (type dash))
-  )
   (wire (pts (xy 283.21 55.88) (xy 283.21 52.07))
     (stroke (width 0) (type default))
@@
     (stroke (width 0) (type default))
   )
+  (polyline (pts (xy 236.855 144.8816) (xy 236.855 241.3))
+    (stroke (width 0.3) (type dash))
+  )
   (wire (pts (xy 337.82 161.29) (xy 337.82 165.1))
     (stroke (width 0) (type default))
@@
     (stroke (width 0) (type default))
   )
-  (polyline (pts (xy 236.855 144.8816) (xy 236.855 241.3))
-    (stroke (width 0.3) (type dash))
-  )
   (wire (pts (xy 54.61 97.79) (xy 54.61 101.6))
     (stroke (width 0) (type default))
   )
+  (polyline (pts (xy 388.5184 33.528) (xy 388.5184 129.9464))
+    (stroke (width 0.3) (type dash))
+  )
   (wire (pts (xy 293.37 113.03) (xy 293.37 116.84))
     (stroke (width 0) (type default))
@@
     (stroke (width 0) (type default))
   )
-  (polyline (pts (xy 237.49 130.175) (xy 28.3464 130.175))
-    (stroke (width 0.3) (type dash))
-  )
   (wire (pts (xy 311.15 83.82) (xy 311.15 86.36))
     (stroke (width 0) (type default))
@@
     (stroke (width 0) (type default))
   )
+  (polyline (pts (xy 28.575 145.5166) (xy 28.575 241.935))
+    (stroke (width 0.3) (type dash))
+  )
   (wire (pts (xy 318.77 93.98) (xy 302.26 93.98))
     (stroke (width 0) (type default))
@@
     (stroke (width 0) (type default))
   )
-  (polyline (pts (xy 388.5184 145.288) (xy 388.5184 241.7064))
-    (stroke (width 0.3) (type dash))
-  )
   (wire (pts (xy 134.62 212.09) (xy 134.62 209.55))
     (stroke (width 0) (type default))
@@
     (stroke (width 0) (type default))
   )
-  (polyline (pts (xy 388.5184 129.9464) (xy 253.0348 129.9464))
-    (stroke (width 0.3) (type dash))
-  )
   (wire (pts (xy 302.26 49.53) (xy 302.26 55.88))
     (stroke (width 0) (type default))
@@
     (stroke (width 0) (type default))
   )
-  (polyline (pts (xy 253.0348 145.3896) (xy 253.0348 241.808))
-    (stroke (width 0.3) (type dash))
-  )
   (wire (pts (xy 58.42 64.77) (xy 58.42 69.85))
     (stroke (width 0) (type default))
@@
     (stroke (width 0) (type default))
   )
+  (polyline (pts (xy 236.855 241.3) (xy 28.575 241.3))
+    (stroke (width 0.3) (type dash))
+  )
   (wire (pts (xy 287.02 49.53) (xy 302.26 49.53))
     (stroke (width 0) (type default))
@@
     (stroke (width 0) (type default))
   )
-  (polyline (pts (xy 388.5184 33.528) (xy 388.5184 129.9464))
-    (stroke (width 0.3) (type dash))
-  )
   (wire (pts (xy 129.54 66.04) (xy 129.54 74.93))
     (stroke (width 0) (type default))
@@
     (stroke (width 0) (type default))
   )
+  (polyline (pts (xy 253.0348 33.528) (xy 388.5184 33.528))
+    (stroke (width 0.3) (type dash))
+  )
   (wire (pts (xy 186.69 190.5) (xy 184.15 190.5))
     (stroke (width 0) (type default))
@@
     (stroke (width 0) (type default))
   )
-  (polyline (pts (xy 388.5184 241.7064) (xy 253.0348 241.7064))
-    (stroke (width 0.3) (type dash))
-  )
   (wire (pts (xy 143.51 66.04) (xy 143.51 69.85))
     (stroke (width 0) (type default))
@@
     (pin "2")
   )
+  (symbol (lib_id "power:GND") (at 144.145 177.8 0) (unit 1)
+    (in_bom yes) (on_board yes)
+    (default_instance (reference "#PWR") (unit 1) (value "GND") (footprint ""))
+    (property "Reference" "#PWR" (id 0) (at 144.145 184.15 0)
+      (effects (font (size 1.27 1.27)) hide)
+    )
+    (property "Value" "GND" (id 1) (at 146.685 181.61 0)
+      (effects (font (size 1.27 1.27)))
+    )
+    (property "Footprint" "" (id 2) (at 144.145 177.8 0)
+      (effects (font (size 1.27 1.27)) hide)
+    )
+    (property "Datasheet" "" (id 3) (at 144.145 177.8 0)
+      (effects (font (size 1.27 1.27)) hide)
+    )
+    (pin "1")
+  )
   (symbol (lib_id "power:GND") (at 359.41 203.2 0) (unit 1)
     (in_bom yes) (on_board yes)
@@
       (reference "#PWR013") (unit 1) (value "GND") (footprint "")
     )
+    (path "/492a51e2-f5d2-42a6-b00f-eb5e4d25143f"
+      (reference "#PWR014") (unit 1) (value "GND") (footprint "")
+    )
     (path "/d7fe01a2-9562-44de-b292-e2eaecfe413e"

Commit message: editor config
Parts:
- C1, C4, C5, C8, C9: renamed from C; value C -> 1uF; footprint (none) -> Capacitor_SMD:C_0603_1608Metric
- C10, C11, C6, C7: renamed from C; value C -> 22nF; footprint (none) -> Capacitor_SMD:C_0603_1608Metric
- C12, C13, C2: renamed from C; value C -> 10uF; footprint (none) -> Capacitor_SMD:C_0603_1608Metric
- C14, C15: renamed from C; value C_Polarized -> 22uF; footprint (none) -> Capacitor_SMD:CP_Elec_4x4.5
- C3: renamed from C; value C -> 100nF; footprint (none) -> Capacitor_SMD:C_0603_1608Metric
- D1: renamed from D; footprint (none) -> LED_SMD:LED_0603_1608Metric
- F1: renamed from F; footprint (none) -> Fuse:Fuse_0603_1608Metric
- FB1, FB2, FB3, FB4, FB5, FB6: renamed from FB; footprint (none) -> Resistor_SMD:R_0603_1608Metric
- FB7, FB8: renamed from FB; value FerriteBead -> DNP; footprint (none) -> Resistor_SMD:R_0603_1608Metric
- H1, H2, H3, H4: renamed from H; footprint (none) -> MountingHole:MountingHole_2.2mm_M2
- J1: renamed from J; value Conn_01x02 -> POWER; footprint (none) -> Connector_PinHeader_2.54mm:PinHeader_1x02_P2.54mm_Vertical
- J2: renamed from J; value Conn_01x06 -> INPUT; footprint (none) -> Connector_JST:JST_SH_SM06B-SRSS-TB_1x06-1MP_P1.00mm_Horizontal
- J3: renamed from J; value Conn_01x04 -> I2C; footprint (none) -> Connector_JST:JST_SH_SM04B-SRSS-TB_1x04-1MP_P1.00mm_Horizontal
- J4: renamed from J; value Conn_01x04 -> UART; footprint (none) -> Connector_JST:JST_SH_SM04B-SRSS-TB_1x04-1MP_P1.00mm_Horizontal
- J5: renamed from J; value Conn_02x03_Odd_Even -> TagConnect; footprint (none) -> loco:Tag-Connect_TC2030-IDC-NL_2x03_P1.27mm_Vertical
- J6: renamed from J; value Conn_01x06 -> GPIO_A; footprint (none) -> Connector_JST:JST_SH_SM06B-SRSS-TB_1x06-1MP_P1.00mm_Horizontal
- J7: renamed from J; value Conn_01x06 -> GPIO_B; footprint (none) -> Connector_JST:JST_SH_SM06B-SRSS-TB_1x06-1MP_P1.00mm_Horizontal
- J8: renamed from J; value Conn_01x04 -> Motor1; footprint (none) -> Connector_JST:JST_SH_SM04B-SRSS-TB_1x04-1MP_P1.00mm_Horizontal
- J9: renamed from J; value Conn_01x04 -> Motor2; footprint (none) -> Connector_JST:JST_SH_SM04B-SRSS-TB_1x04-1MP_P1.00mm_Horizontal
- R1, R11, R12, R24, R26, R4: renamed from R; value R -> 10KΩ; footprint (none) -> Resistor_SMD:R_0603_1608Metric
- R10, R13, R14, R15, R16, R21, R22, R23, R25, R29, R30, R33, R34, R5, R7, R8, R9: renamed from R; value R -> DNP; footprint (none) -> Resistor_SMD:R_0603_1608Metric
- R17, R19: renamed from R; value R -> 15KΩ; footprint (none) -> Resistor_SMD:R_0603_1608Metric
- R18, R20, R27, R28, R6: renamed from R; value R -> 1KΩ; footprint (none) -> Resistor_SMD:R_0603_1608Metric
- R2, R3: renamed from R; value R -> 4.7KΩ; footprint (none) -> Resistor_SMD:R_0603_1608Metric
- R31, R32: renamed from R; value R -> 47KΩ; footprint (none) -> Resistor_SMD:R_0603_1608Metric
- R35, R36, R37, R38: renamed from R; value R -> 0.3Ω; footprint (none) -> Resistor_SMD:R_1206_3216Metric
- RN1, RN2, RN4, RN5: renamed from RN; value R_Pack04 -> 180Ω; footprint (none) -> Resistor_SMD:R_Array_Convex_4x0603
- RN3: renamed from RN; value R_Pack04 -> 10KΩ; footprint (none) -> Resistor_SMD:R_Array_Convex_4x0603
- U2: renamed from U; footprint Package_DFN_QFN:UFQFPN-32-1EP_5x5mm_P0.5mm_EP3.5x3.5mm_ThermalVias -> Package_DFN_QFN:UFQFPN-32-1EP_5x5mm_P0.5mm_EP3.5x3.5mm
- renumbered U to U1, U to U3, U to U4, U to U5

Commit message: pcb rev.0x03
Parts:
- removed C14, C15: 22uF, Capacitor_SMD:CP_Elec_4x4.5, symbol Device:C_Polarized
- removed C4, C9: 1uF, Capacitor_SMD:C_0603_1608Metric, symbol Device:C
- removed C7: 22nF, Capacitor_SMD:C_0603_1608Metric, symbol Device:C
- removed D1: LED, LED_SMD:LED_0603_1608Metric, symbol Device:LED
- removed F1: Polyfuse, Fuse:Fuse_0603_1608Metric, symbol Device:Polyfuse
- removed FB1, FB2, FB3, FB4, FB5, FB6: FerriteBead, Resistor_SMD:R_0603_1608Metric, symbol Device:FerriteBead
- removed FB7, FB8: DNP, Resistor_SMD:R_0603_1608Metric, symbol Device:FerriteBead
- removed J1: POWER, Connector_PinHeader_2.54mm:PinHeader_1x02_P2.54mm_Vertical, symbol Connector_Generic:Conn_01x02
- removed J2: INPUT, Connector_JST:JST_SH_SM06B-SRSS-TB_1x06-1MP_P1.00mm_Horizontal, symbol Connector_Generic:Conn_01x06
- removed J6: GPIO_A, Connector_JST:JST_SH_SM06B-SRSS-TB_1x06-1MP_P1.00mm_Horizontal, symbol Connector_Generic:Conn_01x06
- removed J7: GPIO_B, Connector_JST:JST_SH_SM06B-SRSS-TB_1x06-1MP_P1.00mm_Horizontal, symbol Connector_Generic:Conn_01x06
- removed J8: Motor1, Connector_JST:JST_SH_SM04B-SRSS-TB_1x04-1MP_P1.00mm_Horizontal, symbol Connector_Generic:Conn_01x04
- removed J9: Motor2, Connector_JST:JST_SH_SM04B-SRSS-TB_1x04-1MP_P1.00mm_Horizontal, symbol Connector_Generic:Conn_01x04
- removed R7: DNP, Resistor_SMD:R_0603_1608Metric, symbol Device:R
- removed RN4, RN5: 180Ω, Resistor_SMD:R_Array_Convex_4x0603, symbol Device:R_Pack04
- removed U1: NCV8718, Package_DFN_QFN:DFN-6-1EP_2x2mm_P0.65mm_EP1x1.6mm, symbol loco:NCV8718
- removed U2: STM32G041K8U, Package_DFN_QFN:UFQFPN-32-1EP_5x5mm_P0.5mm_EP3.5x3.5mm, symbol loco:STM32G041K8U
- removed U3: M95512-DRMF3TGK, Package_DFN_QFN:WDFN-8-1EP_3x2mm_P0.5mm_EP1.3x1.4mm, symbol loco:M95512-DRMF3TGK
- removed U5: STSPIN220, Package_DFN_QFN:VQFN-16-1EP_3x3mm_P0.5mm_EP1.8x1.8mm, symbol Driver_Motor:STSPIN220
- added C14, C15, C27, C29, C30, C31: 22nF, Capacitor_SMD:C_0603_1608Metric, symbol Device:C
- added C16, C17, C18, C19, C20, C22, C24, C25, C26, C28, C3: 10uF, Capacitor_SMD:C_0603_1608Metric, symbol Device:C
- added C21, C23, C7, C9: 22uF, Capacitor_SMD:CP_Elec_4x4.5, symbol Device:C_Polarized
- added J10, J14, J15: Stepper1, Connector_JST:JST_PH_B4B-PH-K_1x04_P2.00mm_Vertical, symbol Connector_Generic:Conn_01x04
- added J11: Motor2, Connector_JST:JST_PH_B2B-PH-K_1x02_P2.00mm_Vertical, symbol Connector_Generic:Conn_01x02
- added J12: PWR1, Connector_JST:JST_PH_B2B-PH-K_1x02_P2.00mm_Vertical, symbol Connector_Generic:Conn_01x02
- added J13: PWR2, Connector_JST:JST_PH_B2B-PH-K_1x02_P2.00mm_Vertical, symbol Connector_Generic:Conn_01x02
- added J2: EXT, Connector_JST:JST_PH_B2B-PH-K_1x02_P2.00mm_Vertical, symbol Connector_Generic:Conn_01x02
- added J3: GPIO, Library:Header_03x06_P2.54mm_Vertical, symbol Connector_Generic:Conn_01x08
- added J6: USB_C_Receptacle_USB2.0, @jb:USB_C_Receptacle_JAE_DX07S016JA3R1500, symbol @jb:USB_C_Receptacle_USB2.0
- added J9: Motor1, Connector_JST:JST_PH_B2B-PH-K_1x02_P2.00mm_Vertical, symbol Connector_Generic:Conn_01x02
- added R39, R40, R41, R42, R43: DNP, Resistor_SMD:R_0603_1608Metric, symbol Device:R
- added R4: 5.1KΩ, Resistor_SMD:R_0603_1608Metric, symbol Device:R
- added R44, R48, R49, R52, R53, R59, R61: 10KΩ, Resistor_SMD:R_0603_1608Metric, symbol Device:R
- added R45, R46, R50, R51: 0.3Ω, Resistor_SMD:R_1206_3216Metric, symbol Device:R
- added R47: 150KΩ, Resistor_SMD:R_0603_1608Metric, symbol Device:R
- added R54, R56: 47KΩ, Resistor_SMD:R_0603_1608Metric, symbol Device:R
- added R55, R57, R58, R60: 1KΩ, Resistor_SMD:R_0603_1608Metric, symbol Device:R
- added U1: LD1117S33TR_SOT223, Package_TO_SOT_SMD:SOT-223-3_TabPin2, symbol Regulator_Linear:LD1117S33TR_SOT223
- added U2: STM32C031CxUx, Package_QFP:LQFP-48_7x7mm_P0.5mm, symbol @jb:STM32C031CxUx
- added U3: STSPIN240, Package_DFN_QFN:VQFN-16-1EP_3x3mm_P0.5mm_EP1.8x1.8mm, symbol Driver_Motor:STSPIN240
- added U5, U6, U7: AP22652_3x, Package_TO_SOT_SMD:SOT-23-6, symbol @jb:AP22652_3x
- added U8, U9: STSPIN220, Package_DFN_QFN:VQFN-16-1EP_3x3mm_P0.5mm_EP1.8x1.8mm, symbol Driver_Motor:STSPIN220
- C11, C6: value 22nF -> 10uF
- C12: value 10uF -> 22nF
- C4: renamed from C1; value 1uF -> 10uF
- C8: value 1uF -> 10uF
- H1, H2, H3, H4: footprint MountingHole:MountingHole_2.2mm_M2 -> MountingHole:MountingHole_3.2mm_M3_Pad_Via
- J1: renamed from J3; footprint Connector_JST:JST_SH_SM04B-SRSS-TB_1x04-1MP_P1.00mm_Horizontal -> Connector_JST:JST_SH_BM04B-SRSS-TB_1x04-1MP_P1.00mm_Vertical
- J7: renamed from J4; footprint Connector_JST:JST_SH_SM04B-SRSS-TB_1x04-1MP_P1.00mm_Horizontal -> Connector_JST:JST_SH_BM04B-SRSS-TB_1x04-1MP_P1.00mm_Vertical
- J8: renamed from J5; footprint loco:Tag-Connect_TC2030-IDC-NL_2x03_P1.27mm_Vertical -> Connector:Tag-Connect_TC2030-IDC-NL_2x03_P1.27mm_Vertical
- R1, R11: value 10KΩ -> DNP
- R12: value 10KΩ -> 0.3Ω; footprint Resistor_SMD:R_0603_1608Metric -> Resistor_SMD:R_1206_3216Metric
- R13, R16: value DNP -> 0.3Ω; footprint Resistor_SMD:R_0603_1608Metric -> Resistor_SMD:R_1206_3216Metric
- R14, R15, R25: value DNP -> 10KΩ
- R17: value 15KΩ -> 0.3Ω; footprint Resistor_SMD:R_0603_1608Metric -> Resistor_SMD:R_1206_3216Metric
- R18, R27, R28: value 1KΩ -> 10KΩ
- R19: value 15KΩ -> 10KΩ
- R20: value 1KΩ -> 47KΩ
- R21, R23: value DNP -> 1KΩ
- R22: value DNP -> 47KΩ
- R24, R26: value 10KΩ -> 1KΩ
- R29: value DNP -> 0Ω
- R31: value 47KΩ -> 10KΩ
- R32: value 47KΩ -> 0Ω
- R34: value DNP -> 150KΩ
- R35: value 0.3Ω -> 150KΩ; footprint Resistor_SMD:R_1206_3216Metric -> Resistor_SMD:R_0603_1608Metric
- R36, R37, R38: value 0.3Ω -> DNP; footprint Resistor_SMD:R_1206_3216Metric -> Resistor_SMD:R_0603_1608Metric
- R5: value DNP -> 5.1KΩ
- R6: value 1KΩ -> DNP
- RN1, RN2: value 180Ω -> 190Ω
- RN3: value 10KΩ -> 190Ω
- renumbered C2 to C1, C3 to C2, R4 to R7
Connections:
- net M2S1 is gone; now on net GND: R37.2
- net M2S2 is gone; now on an unnamed net: R38.2
- net M2_EN is gone; now on net GND: R12.1
- net GND: now also R16.1, R17.1, R22.2, R24.2, R25.2, R26.2, R27.2, R34.1, R5.1, R8.1, R9.2, C14.2, C15.2, C16.2, C17.2, C18.2, C19.2, C20.2, C21.2, C22.2, C23.2, C24.2, C25.2, C26.2, C27.2, C28.2, C29.2, C3.2, C30.2, C31.2, C7.2, C9.2, J12.1 (Pin_1), J13.1 (Pin_1), J2.1 (Pin_1), J3.8 (Pin_8), J6.A1 (GND), R4.2, R40.1, R41.2, R45.1, R46.1, R47.1, R50.1, R51.1, R54.2, R56.2, R58.2, R59.2, R60.2, R61.2, U1.1 (GND), U2.7 (VSS), U3.17 (EPAD), U3.7 (GND), U5.2 (GND), U6.2 (GND), U7.2 (GND), U8.17 (EPAD), U8.7 (GND), U9.17 (EPAD), U9.7 (GND); no longer R10.1, R14.1, R18.2, R21.1, R22.1, R29.1, R30.1, R31.2, R32.2, R37.1, R38.1, R9.1, RN3.6 (R3.2)
- net GPIO1: now also RN1.7 (R2.2), U2.11 (PA0)
- net GPIO2: now also RN1.6 (R3.2), U2.12 (PA1)
- net GPIO3: now also RN1.5 (R4.2), U2.13 (PA2)
- net GPIO4: now also RN3.8 (R1.2), U2.14 (PA3)
- net GPIO5: now also RN3.7 (R2.2), U2.15 (PA4)
- net GPIO6: now also RN3.6 (R3.2), U2.16 (PA5)
- net I2C_SCL: now also RN2.2 (R2.1), U2.47 (PB8); no longer RN2.7 (R2.2)
- net I2C_SDA: now also RN2.1 (R1.1), U2.48 (PB9); no longer RN2.8 (R1.2)
- net RESET: now also U2.8 (PF0)
- net UART_RX: now also RN2.3 (R3.1), U2.46 (PB7); no longer RN2.5 (R4.2)
- net UART_TX: now also RN2.4 (R4.1), U2.45 (PB6); no longer RN2.6 (R3.2)
- net VCC: now also C6.1, C8.1, R10.1, R11.2, R30.2, R33.2, R38.1, C20.1, C21.1, C22.1, C23.1, C7.1, C9.1, J2.2 (Pin_2), J6.A4 (VBUS), J6.A9 (VBUS), R39.2, R42.1, R43.2, U1.3 (VI), U3.6 (VS), U8.6 (VS), U9.6 (VS); no longer C12.1, C13.1, R1.1
- net VDD: now also R28.1, R29.1, R31.1, R32.1, C24.1, C3.1, R44.1, U1.2 (VO), U2.5 (VREF+), U2.6 (VDD), U7.1 (VIN); no longer R15.2, R16.2, R17.2, R19.2, R23.2, R24.1, R25.2, R26.1, R33.2, R34.2, R6.1, R8.2, RN3.7 (R2.2), RN3.8 (R1.2)
- net at R10.2: now also R8.2, U4.15 (MODE2); no longer R8.1
- net M_FAULT: now reaches R14.2
- net M_FAULT: now also C10.1, U2.40 (PD2), U3.13 (EN/FLT); no longer R16.1
- net GPIO_PWR : now reaches R6.2
- net GPIO_PWR : now also R1.2, C25.1, J3.7 (Pin_7), U7.6 (VOUT)
- net at R20.1: now also R21.1, U3.12 (TOFF); no longer R19.1
- net S1_STBY: now reaches U4.14 (STBY/RESET)
- net S1_STBY: now also R27.1, U2.44 (PB5); no longer R24.2
- net at RN3.3 (R3.1): now also J3.6 (Pin_6); no longer R5.1
- net at J1.3 (Pin_3), R3.2: now also RN2.8 (R1.2); no longer RN2.1 (R1.1)
- net at J1.4 (Pin_4), R2.2: now also RN2.7 (R2.2); no longer RN2.2 (R2.1)
- net at C11.1: now also R18.2, R24.1, U3.11 (REF); no longer R28.2
- net at RN3.1 (R1.1): now also J3.4 (Pin_4)
- net at RN3.2 (R2.1): now also J3.5 (Pin_5)
- net at J7.3 (Pin_3): now also RN2.5 (R4.2); no longer RN2.3 (R3.1)
- net at J7.4 (Pin_4): now also RN2.6 (R3.2); no longer RN2.4 (R4.1)
- net BTN1: no longer names the net of RN1.4 (R4.1)
- net BTN1: now also J3.3 (Pin_3)
- net BTN2: no longer names the net of RN1.3 (R3.1)
- net BTN2: now also J3.2 (Pin_2)
- net ENC1: no longer names the net of RN1.1 (R1.1)
- net ENC2: no longer names the net of RN1.2 (R2.1)
- net ENC2: now also J3.1 (Pin_1)
- net I2C_VDD: no longer names the net of J1.2 (Pin_2)
- net I2C_VDD: now also R1.1
- net M1A1 renamed S1_A1
- net S1_A1: now also J10.1 (Pin_1)
- net M1A2 renamed S1_A2
- net S1_A2: now also J10.2 (Pin_2)
- net M1B1 renamed S1_B1
- net S1_B1: now also J10.4 (Pin_4)
- net M1B2 renamed S1_B2
- net S1_B2: now also J10.3 (Pin_3)
- net M1S1: no longer names the net of R35.2
- net M1S1: now also U6.5 (ILIM); no longer U4.4 (SENSEA)
- net M1S2: no longer names the net of R36.2
- net M1S2: now also U8.15 (MODE2); no longer U4.9 (SENSEB)
- removed net M1_DIR: R29.2, R33.1, U4.1 (DIR)
- net M1_EN: no longer names the net of R11.1
- net M1_EN: now also R9.1, U4.16 (MODE1)
- removed net M1_FLT: C6.1, R11.2, U4.13 (EN/FLT)
- removed net M1_STCK: R21.2, R23.1, U4.2 (STCK)
- removed net M2_DIR: R30.2, R34.1
- net M2_FLT renamed M_S1
- net M_S1: now also U3.4 (SENSEA)
- net M2_STCK renamed M_STBY
- net M_STBY: now also U2.38 (PD0), U3.14 (STBY/RESET); no longer R22.2
- net SWDCLK: no longer names the net of J8.4 (Pin_4)
- net SWDCLK: now also U2.36 (PA14)
- net SWDIO: no longer names the net of R5.2
- net SWDIO: now also J6.A5 (CC1); no longer J8.2 (Pin_2)
- net UART_VDD: no longer names the net of J7.2 (Pin_2)
- net UART_VDD: now also R6.1
- new net: J8.2 (Pin_2), U2.35 (PA13)
- new net: C18.1, J12.2 (Pin_2), U5.6 (VOUT)
- new net: C28.1, R53.2, R60.1, U9.11 (REF)
- new net: R40.2, R42.2, U9.15 (MODE2)
- new net: R41.1, R43.1, U9.16 (MODE1)
- new net: C13.1, R19.2, R26.1, U4.11 (REF)
- new net: C17.1, R29.2, R30.1, U6.1 (VIN)
- new net: J6.B5 (CC2), R4.1
- new net: R34.2, U5.5 (ILIM)
- new net: R22.1, R23.1, U4.12 (TOFF)
- new net: C15.1, R23.2
- new net: C12.1, R21.2
- new net: R47.2, U7.5 (ILIM)
- new net: R37.1, R39.1, U8.16 (MODE1)
- new net: R56.1, R57.1, U9.12 (TOFF)
- new net: C31.1, R57.2
- new net: C26.1, R52.2, R58.1, U8.11 (REF)
- new net: C19.1, J13.2 (Pin_2), U6.6 (VOUT)
- new net: C16.1, R32.2, R33.1, U5.1 (VIN)
- new net: R54.1, R55.1, U8.12 (TOFF)
- new net: C30.1, R55.2
- new net GPIO_PWR_SENSE: R44.2, U2.3 (PC15), U7.4 (FAULT)
- new net GPIO_PWR_SWITCH: U2.4 (PF3), U7.3 (EN)
- new net M1_PHASE: U2.34 (PA12), U3.1 (PHA)
- new net M1_PWM: U2.32 (PA10), U3.2 (PWMA)
- new net M2_PHASE: U2.37 (PA15), U3.15 (PHB)
- new net M2_PWM: U2.33 (PA11), U3.16 (PWMB)
- new net M_A1: J9.1 (Pin_1), U3.3 (OUTA1)
- new net M_A2: J9.2 (Pin_2), U3.5 (OUTA2)
- new net M_B1: J11.2 (Pin_2), U3.10 (OUTB1)
- new net M_B2: J11.1 (Pin_1), U3.8 (OUTB2)
- new net M_EN: R14.1, U2.39 (PD1)
- new net M_REF: R18.1, U2.43 (PB4)
- new net M_S2: R16.2, U3.9 (SENSEB)
- new net PWR1_SENSE: R31.2, U2.23 (PB11), U5.4 (FAULT)
- new net PWR1_SWITCH: U2.24 (PB12), U5.3 (EN)
- new net PWR2_SENSE: R28.2, U2.9 (PF1), U6.4 (FAULT)
- new net PWR2_SWITCH: U2.10 (PF2), U6.3 (EN)
- new net S1_DIR: U2.42 (PB3), U4.1 (DIR)
- new net S1_EN: R15.1, U2.2 (PC14)
- new net S1_FAULT: C14.1, R15.2, U2.1 (PC13), U4.13 (EN/FLT)
- new net S1_REF: R19.1, U2.31 (PC7)
- new net S1_S1: R13.2, U4.4 (SENSEA)
- new net S1_S2: R17.2, U4.9 (SENSEB)
- new net S1_STEP: U2.41 (PD3), U4.2 (STCK)
- new net S2_A1: J14.1 (Pin_1), U8.3 (OUTA1)
- new net S2_A2: J14.2 (Pin_2), U8.5 (OUTA2)
- new net S2_B1: J14.4 (Pin_4), U8.10 (OUTB1)
- new net S2_B2: J14.3 (Pin_3), U8.8 (OUTB2)
- new net S2_DIR: U2.18 (PA7), U8.1 (DIR)
- new net S2_EN: R48.1, U2.21 (PB2)
- new net S2_FAULT: C27.1, R48.2, U2.22 (PB10), U8.13 (EN/FLT)
- new net S2_REF: R52.1, U2.20 (PB1)
- new net S2_S1: R45.2, U8.4 (SENSEA)
- new net S2_S2: R50.2, U8.9 (SENSEB)
- new net S2_STBY: R59.1, U2.19 (PB0), U8.14 (STBY/RESET)
- new net S2_STEP: U2.17 (PA6), U8.2 (STCK)
- new net S3_A1: J15.1 (Pin_1), U9.3 (OUTA1)
- new net S3_A2: J15.2 (Pin_2), U9.5 (OUTA2)
- new net S3_B1: J15.4 (Pin_4), U9.10 (OUTB1)
- new net S3_B2: J15.3 (Pin_3), U9.8 (OUTB2)
- new net S3_DIR: U2.25 (PB13), U9.1 (DIR)
- new net S3_EN: R49.1, U2.29 (PA9)
- new net S3_FAULT: C29.1, R49.2, U2.30 (PC6), U9.13 (EN/FLT)
- new net S3_REF: R53.1, U2.28 (PA8)
- new net S3_S1: R46.2, U9.4 (SENSEA)
- new net S3_S2: R51.2, U9.9 (SENSEB)
- new net S3_STBY: R61.1, U2.27 (PB15), U9.14 (STBY/RESET)
- new net S3_STEP: U2.26 (PB14), U9.2 (STCK)
- no-connect marks 3 -> 12
Other:
- note added: "DC Motor Driver"
- note added: "External Power"
- note added: "GPIO"
- note added: "Power"
- note added: "Stepper Driver 1"
- note added: "Stepper Driver 2"
- note added: "Stepper Driver 3"
- note removed: "Power & Connectors"
- note removed: "Stepper Motor Channel 1"
- note removed: "Stepper Motor Channel 2"
- moved on the sheet: C1, C2, C4, C5, H1, J1, J7, J8, R2, R3, R7, RN2
