File: pcb/loco.kicad_sch (KiCad schematic)
At the start: 121 parts, among them J1 I2C, J10 Stepper1, J11 Motor2, J12 PWR1, J13 PWR2, J14 Stepper1, J15 Stepper1, J2 EXT, J3 GPIO, J6 USB_C_Receptacle_USB2.0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

Commit message: rev 0x04
Connections:
- net PWR2_SENSE: now also U2.8 (PF0); no longer U2.9 (PF1)
- net PWR2_SWITCH: now also U2.9 (PF1); no longer U2.10 (PF2)
- net RESET: now also U2.10 (PF2); no longer U2.8 (PF0)
Changed lines of the file:
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@@
   (title_block
     (title "loco")
-    (date "2023-02-04")
-    (rev "0x03")
+    (date "2023-02-18")
+    (rev "0x04")
     (company "vitaly.codes")
   )
@@
     (effects (font (size 1.27 1.27)) (justify right bottom))
   )
-  (label "PWR2_SENSE" (at 316.23 52.07 180) (fields_autoplaced)
+  (label "PWR2_SENSE" (at 316.23 49.53 180) (fields_autoplaced)
     (effects (font (size 1.27 1.27)) (justify right bottom))
   )
@@
     (effects (font (size 1.27 1.27)) (justify left bottom))
   )
-  (label "PWR2_SWITCH" (at 316.23 54.61 180) (fields_autoplaced)
+  (label "PWR2_SWITCH" (at 316.23 52.07 180) (fields_autoplaced)
     (effects (font (size 1.27 1.27)) (justify right bottom))
   )
@@
     (effects (font (size 1.27 1.27)) (justify left bottom))
   )
-  (label "RESET" (at 316.23 49.53 180) (fields_autoplaced)
+  (label "RESET" (at 316.23 54.61 180) (fields_autoplaced)
     (effects (font (size 1.27 1.27)) (justify right bottom))
   )
